File: cad/data-logger.kicad_pcb (KiCad board)
At the start: 2 copper layers, 57.2 x 27.9 mm, 29 parts, among them IC1 TP4054-42-SOT25-R, J1 Micro_SD_Card, J2 Conn_01x02, J3 Conn_01x02, J4 Conn_01x08, J5 Conn_01x08, U1 ATMEGA328-AU, U2 MCP1700-3302E_SOT23, U3 DS1307Z+, Y1 Crystal_GND24_Small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

Commit message: Update kicad schematic and layout files to support kicad 7
Other:
- net class Default removed
